File: Hardware/Eagle/2020-03-08 LN2 Autofill Controller.sch (EAGLE design)
At the start: 28 parts, among them SW1 SWITCH-OMRON-B3J-1LED, SW2 SWITCH-OMRON-B3J-1LED, SW3 SWITCH-OMRON-B3J-1LED, SW4 SWITCH-OMRON-B3J-1LED, U1 MC14490DWG, U3 ISO7421DR

Commit message: Switched to a right angle connector on the RJ11 breakout
Parts:
- JP3: value Molex 0022292021 -> Molex 22112022
- SW1, SW2, SW3, SW4: value SWITCH-OMRON-B3J-1LED -> Omron B3J-2100
Other:
- note added: "Rewire for RJ11 6-pin breakout"
- note added: "Switch to stand-up version"
Changed lines of the file:
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@@
 <parts>
 <part name="JP2" library="AUmlib" library_urn="urn:adsk.eagle:library:9166017" deviceset="PINHD-1X20" device="" package3d_urn="urn:adsk.eagle:package:22441/2"/>
-<part name="SW1" library="AUmlib" library_urn="urn:adsk.eagle:library:9166017" deviceset="SWITCH-OMRON-B3J-1LED" device="" package3d_urn="urn:adsk.eagle:package:16346131/2"/>
-<part name="SW2" library="AUmlib" library_urn="urn:adsk.eagle:library:9166017" deviceset="SWITCH-OMRON-B3J-1LED" device="" package3d_urn="urn:adsk.eagle:package:16346131/2"/>
-<part name="SW3" library="AUmlib" library_urn="urn:adsk.eagle:library:9166017" deviceset="SWITCH-OMRON-B3J-1LED" device="" package3d_urn="urn:adsk.eagle:package:16346131/2"/>
-<part name="SW4" library="AUmlib" library_urn="urn:adsk.eagle:library:9166017" deviceset="SWITCH-OMRON-B3J-1LED" device="" package3d_urn="urn:adsk.eagle:package:16346131/2"/>
+<part name="SW1" library="AUmlib" library_urn="urn:adsk.eagle:library:9166017" deviceset="SWITCH-OMRON-B3J-1LED" device="" package3d_urn="urn:adsk.eagle:package:16346131/2" value="Omron B3J-2100"/>
+<part name="SW2" library="AUmlib" library_urn="urn:adsk.eagle:library:9166017" deviceset="SWITCH-OMRON-B3J-1LED" device="" package3d_urn="urn:adsk.eagle:package:16346131/2" value="Omron B3J-2100"/>
+<part name="SW3" library="AUmlib" library_urn="urn:adsk.eagle:library:9166017" deviceset="SWITCH-OMRON-B3J-1LED" device="" package3d_urn="urn:adsk.eagle:package:16346131/2" value="Omron B3J-2100"/>
+<part name="SW4" library="AUmlib" library_urn="urn:adsk.eagle:library:9166017" deviceset="SWITCH-OMRON-B3J-1LED" device="" package3d_urn="urn:adsk.eagle:package:16346131/2" value="Omron B3J-2100"/>
 <part name="CNANO1" library="AUmlib" library_urn="urn:adsk.eagle:library:9166017" deviceset="CURIOSITYNANO4809" device="CASTELLATED" package3d_urn="urn:adsk.eagle:package:15461731/6"/>
 <part name="VR1" library="AUmlib" library_urn="urn:adsk.eagle:library:9166017" deviceset="OKI-78SR" device="" package3d_urn="urn:adsk.eagle:package:23154151/4" value="OKI-78SR-5"/>
@@
 <part name="GND13" library="AUmlib" library_urn="urn:adsk.eagle:library:9166017" deviceset="GND" device=""/>
 <part name="EN1" library="AUmlib" library_urn="urn:adsk.eagle:library:9166017" deviceset="ENC-BOURNES-PEC11L" device="" package3d_urn="urn:adsk.eagle:package:16443896/3" value="PEC11L-4120F-S0020"/>
-<part name="JP3" library="AUmlib" library_urn="urn:adsk.eagle:library:9166017" deviceset="PINHD-1X2" device="MOLEX-02-VERT" package3d_urn="urn:adsk.eagle:package:16444314/3" value="Molex 0022292021"/>
+<part name="JP3" library="AUmlib" library_urn="urn:adsk.eagle:library:9166017" deviceset="PINHD-1X2" device="MOLEX-02-VERT" package3d_urn="urn:adsk.eagle:package:16444314/3" value="Molex 22112022"/>
 <part name="U3" library="AUmlib" library_urn="urn:adsk.eagle:library:9166017" deviceset="ISO7421DR" device="TI-SOIC-D8" package3d_urn="urn:adsk.eagle:package:16444440/1" value="ISO7421DR"/>
 <part name="U1" library="AUmlib" library_urn="urn:adsk.eagle:library:9166017" deviceset="DEBOUNCER-MC14490DWG" device="SOIC-16-WB" package3d_urn="urn:adsk.eagle:package:16444518/1" value="MC14490DWG"/>
@@
 <wire x1="304.8" y1="180.34" x2="243.84" y2="180.34" width="0.254" layer="250"/>
 <wire x1="243.84" y1="180.34" x2="243.84" y2="233.68" width="0.254" layer="250"/>
+<text x="7.62" y="187.96" size="1.778" layer="250">Rewire for RJ11 6-pin breakout</text>
+<text x="7.62" y="86.36" size="1.778" layer="250">Switch to stand-up version</text>
 </plain>
 <instances>

Commit message: Swapped 5VDC convert to stand-up version
Parts:
- removed VR1: OKI-78SR-5, AUmlib:OKI-78SR
- added PS2: OKI-78SR-5/1.5-W36-C, AUmlib:OKI-78SR-5/1.5-W36-C
Connections:
- new net VOUT: PS2.VOUT
- net +24V: now also PS2.VIN; no longer VR1.VIN
- net +5V: no longer VR1.VOUT
- net GND: now also PS2.GND; no longer VR1.GND
Changed lines of the file:
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@@
 <part name="SW4" library="AUmlib" library_urn="urn:adsk.eagle:library:9166017" deviceset="SWITCH-OMRON-B3J-1LED" device="" package3d_urn="urn:adsk.eagle:package:16346131/2" value="Omron B3J-2100"/>
 <part name="CNANO1" library="AUmlib" library_urn="urn:adsk.eagle:library:9166017" deviceset="CURIOSITYNANO4809" device="CASTELLATED" package3d_urn="urn:adsk.eagle:package:15461731/6"/>
-<part name="VR1" library="AUmlib" library_urn="urn:adsk.eagle:library:9166017" deviceset="OKI-78SR" device="" package3d_urn="urn:adsk.eagle:package:23154151/4" value="OKI-78SR-5"/>
 <part name="C1" library="AUmlib" library_urn="urn:adsk.eagle:library:9166017" deviceset="C-US" device="C1210K" package3d_urn="urn:adsk.eagle:package:4021329/2" value="10uF"/>
 <part name="P+2" library="AUmlib" library_urn="urn:adsk.eagle:library:9166017" deviceset="+24V" device=""/>
@@
 <part name="TP2" library="AUmlib" library_urn="urn:adsk.eagle:library:9166017" deviceset="PINHD-1X1" device="TESTPOINT1" package3d_urn="urn:adsk.eagle:package:15845500/3"/>
 <part name="GND16" library="AUmlib" library_urn="urn:adsk.eagle:library:9166017" deviceset="GND" device=""/>
+<part name="PS2" library="AUmlib" library_urn="urn:adsk.eagle:library:9166017" deviceset="OKI-78SR-5/1.5-W36-C" device="" package3d_urn="urn:adsk.eagle:package:24308288/2"/>
 </parts>
 <sheets>
@@
 <attribute name="VALUE" x="248.92" y="86.36" size="1.778" layer="96"/>
 </instance>
-<instance part="VR1" gate="G$1" x="33.02" y="71.12" smashed="yes">
-<attribute name="NAME" x="24.13" y="77.47" size="1.778" layer="95"/>
-<attribute name="VALUE" x="34.29" y="63.5" size="1.778" layer="96"/>
-</instance>
 <instance part="C1" gate="G$1" x="15.24" y="66.04" smashed="yes">
 <attribute name="NAME" x="11.176" y="66.675" size="1.778" layer="95"/>
@@
 <instance part="GND16" gate="1" x="198.12" y="185.42" smashed="yes">
 <attribute name="VALUE" x="195.58" y="182.88" size="1.778" layer="96"/>
+</instance>
+<instance part="PS2" gate="G$1" x="33.02" y="68.58" smashed="yes">
+<attribute name="NAME" x="30.48" y="74.93" size="1.778" layer="95"/>
+<attribute name="VALUE" x="20.32" y="62.23" size="1.778" layer="96"/>
 </instance>
 </instances>
@@
 <segment>
 <pinref part="GND4" gate="1" pin="GND"/>
-<pinref part="VR1" gate="G$1" pin="GND"/>
 <wire x1="45.72" y1="58.42" x2="45.72" y2="68.58" width="0.1524" layer="91"/>
 <wire x1="45.72" y1="68.58" x2="43.18" y2="68.58" width="0.1524" layer="91"/>
+<pinref part="PS2" gate="G$1" pin="GND"/>
 </segment>
 <segment>
@@
 <wire x1="48.26" y1="127" x2="40.64" y2="127" width="0.1524" layer="91"/>
 <label x="40.64" y="127" size="1.778" layer="95" rot="MR0" xref="yes"/>
-</segment>
-<segment>
-<pinref part="VR1" gate="G$1" pin="VOUT"/>
-<wire x1="43.18" y1="71.12" x2="48.26" y2="71.12" width="0.1524" layer="91"/>
-<pinref part="P+3" gate="1" pin="+5V"/>
-<wire x1="48.26" y1="71.12" x2="48.26" y2="76.2" width="0.1524" layer="91"/>
 </segment>
 <segment>
@@
 <pinref part="C1" gate="G$1" pin="1"/>
 <wire x1="15.24" y1="68.58" x2="15.24" y2="71.12" width="0.1524" layer="91"/>
-<pinref part="VR1" gate="G$1" pin="VIN"/>
 <wire x1="15.24" y1="71.12" x2="22.86" y2="71.12" width="0.1524" layer="91"/>
 <pinref part="P+4" gate="1" pin="+24V"/>
 <wire x1="15.24" y1="71.12" x2="15.24" y2="76.2" width="0.1524" layer="91"/>
 <junction x="15.24" y="71.12"/>
+<pinref part="PS2" gate="G$1" pin="VIN"/>
 </segment>
 </net>
@@
 </segment>
 </net>
+<net name="VOUT" class="0">
+<segment>
+<wire x1="43.18" y1="71.12" x2="48.26" y2="71.12" width="0.1524" layer="91"/>
+<pinref part="P+3" gate="1" pin="+5V"/>
+<wire x1="48.26" y1="71.12" x2="48.26" y2="76.2" width="0.1524" layer="91"/>
+<pinref part="PS2" gate="G$1" pin="VOUT"/>
+</segment>
+</net>

Commit message: Start rewiring
Parts:
- removed TP1: (no value), AUmlib:PINHD-1X1TESTPOINT1
- added TP3: TP5000-TESTPOINT-BLK, AUmlib:TP5000-TESTPOINT-BLK
- TP2: value (none) -> TP5000-TESTPOINT-BLU; device AUmlib:PINHD-1X1TESTPOINT1 -> AUmlib:TP5000-TESTPOINT-BLU
Connections:
- net A1IN: no longer TP1.1
- net GND: now also TP3.1; no longer TP2.1
- net PRES: now also TP2.1
Changed lines of the file:
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@@
 <part name="GND11" library="AUmlib" library_urn="urn:adsk.eagle:library:9166017" deviceset="GND" device=""/>
 <part name="R5" library="AUmlib" library_urn="urn:adsk.eagle:library:9166017" deviceset="R-US_" device="R0805" package3d_urn="urn:adsk.eagle:package:4021199/4" value="270R"/>
-<part name="TP1" library="AUmlib" library_urn="urn:adsk.eagle:library:9166017" deviceset="PINHD-1X1" device="TESTPOINT1" package3d_urn="urn:adsk.eagle:package:15845500/3"/>
-<part name="TP2" library="AUmlib" library_urn="urn:adsk.eagle:library:9166017" deviceset="PINHD-1X1" device="TESTPOINT1" package3d_urn="urn:adsk.eagle:package:15845500/3"/>
 <part name="GND16" library="AUmlib" library_urn="urn:adsk.eagle:library:9166017" deviceset="GND" device=""/>
 <part name="PS2" library="AUmlib" library_urn="urn:adsk.eagle:library:9166017" deviceset="OKI-78SR-5/1.5-W36-C" device="" package3d_urn="urn:adsk.eagle:package:24308288/2"/>
+<part name="TP3" library="AUmlib" library_urn="urn:adsk.eagle:library:9166017" deviceset="TP5000-TESTPOINT-BLK" device="" package3d_urn="urn:adsk.eagle:package:24642442/4"/>
+<part name="TP2" library="AUmlib" library_urn="urn:adsk.eagle:library:9166017" deviceset="TP5000-TESTPOINT-BLU" device="" package3d_urn="urn:adsk.eagle:package:24643711/2"/>
 </parts>
 <sheets>
@@
 <attribute name="VALUE" x="142.24" y="193.802" size="1.778" layer="96" rot="R180"/>
 </instance>
-<instance part="TP1" gate="G$1" x="187.96" y="200.66" smashed="yes" rot="R180">
-<attribute name="NAME" x="194.31" y="197.485" size="1.778" layer="95" rot="R180"/>
-<attribute name="VALUE" x="194.31" y="205.74" size="1.778" layer="96" rot="R180"/>
-</instance>
-<instance part="TP2" gate="G$1" x="187.96" y="190.5" smashed="yes" rot="R180">
-<attribute name="NAME" x="194.31" y="187.325" size="1.778" layer="95" rot="R180"/>
-<attribute name="VALUE" x="194.31" y="195.58" size="1.778" layer="96" rot="R180"/>
-</instance>
-<instance part="GND16" gate="1" x="198.12" y="185.42" smashed="yes">
-<attribute name="VALUE" x="195.58" y="182.88" size="1.778" layer="96"/>
+<instance part="GND16" gate="1" x="297.18" y="187.96" smashed="yes">
+<attribute name="VALUE" x="294.64" y="185.42" size="1.778" layer="96"/>
 </instance>
 <instance part="PS2" gate="G$1" x="33.02" y="68.58" smashed="yes">
 <attribute name="NAME" x="30.48" y="74.93" size="1.778" layer="95"/>
 <attribute name="VALUE" x="20.32" y="62.23" size="1.778" layer="96"/>
+</instance>
+<instance part="TP3" gate="G$1" x="289.56" y="193.04" smashed="yes" rot="R180">
+<attribute name="NAME" x="292.1" y="189.23" size="1.778" layer="95" rot="R180"/>
+<attribute name="VALUE" x="302.26" y="182.88" size="1.778" layer="96" rot="R180"/>
+</instance>
+<instance part="TP2" gate="G$1" x="190.5" y="200.66" smashed="yes" rot="R180">
+<attribute name="NAME" x="193.04" y="196.85" size="1.778" layer="95" rot="R180"/>
+<attribute name="VALUE" x="213.36" y="193.04" size="1.778" layer="96" rot="R180"/>
 </instance>
 </instances>
@@
 </segment>
 <segment>
-<pinref part="TP2" gate="G$1" pin="1"/>
-<wire x1="190.5" y1="190.5" x2="198.12" y2="190.5" width="0.1524" layer="91"/>
 <pinref part="GND16" gate="1" pin="GND"/>
-<wire x1="198.12" y1="190.5" x2="198.12" y2="187.96" width="0.1524" layer="91"/>
+<wire x1="297.18" y1="193.04" x2="297.18" y2="190.5" width="0.1524" layer="91"/>
+<pinref part="TP3" gate="G$1" pin="1"/>
+<wire x1="294.64" y1="193.04" x2="297.18" y2="193.04" width="0.1524" layer="91"/>
 </segment>
 <segment>
@@
 <label x="292.1" y="129.54" size="1.778" layer="95" xref="yes"/>
 </segment>
+<segment>
+<wire x1="195.58" y1="200.66" x2="198.12" y2="200.66" width="0.1524" layer="91"/>
+<label x="198.12" y="200.66" size="1.778" layer="95" xref="yes"/>
+<pinref part="TP2" gate="G$1" pin="1"/>
+</segment>
 </net>
 <net name="N$12" class="0">
@@
 <label x="279.4" y="132.08" size="1.778" layer="95" xref="yes"/>
 </segment>
-<segment>
-<pinref part="TP1" gate="G$1" pin="1"/>
-<wire x1="190.5" y1="200.66" x2="198.12" y2="200.66" width="0.1524" layer="91"/>
-<label x="198.12" y="200.66" size="1.778" layer="95" xref="yes"/>
-</segment>
-</net>
+</net>
