File: Hardware/Eagle/2020-03-08 LN2 Autofill Controller.sch (EAGLE design)
At the start: 28 parts, among them SW1 Omron B3J-2100, SW2 Omron B3J-2100, SW3 Omron B3J-2100, SW4 Omron B3J-2100, U1 MC14490DWG, U3 ISO7421DR

Commit message: Save minor changes?
Connections:
- net N$4 renamed /RES
Changed lines of the file:
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@@
 </segment>
 </net>
-<net name="N$4" class="0">
+<net name="/RES" class="0">
 <segment>
 <pinref part="R5" gate="G$1" pin="1"/>
