File: Hardware/Eagle/LN2 Autofill Connectors.sch (EAGLE design)
At the start: 45 parts, among them J1 Phoenix 1455997, J2 Phoenix 1455997, J3 Phoenix 1455997, J4 Phoenix 1455997, J5 Phoenix 1456116, J6 Phoenix 1456116, J7 Phoenix 1456116, J8 Phoenix 1456116, Q1 RTR030N05HZG, Q2 RTR030N05HZG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

Commit message: Added gate resistor and re-routed connector board
Parts:
- added R25, R26, R27, R28: 100K, AUmlib:R-US_R0805
- JP2, JP3: value (none) -> MOLEX 53822112022
Connections:
- net GNDI: now also R25.1, R26.1, R27.1, R28.1
- net N$1: now also R25.2
- net N$2: now also R26.2
- net N$3: now also R27.2
- net N$4: now also R28.2
Other:
- note added: "LN2 Autofill Connector Board 2021-02-21 Panel connectors to thermistors and solenoid valves"
- note removed: "LN2 Autofill Connector Board 2020-03-07 Panel connectors to thermistors and solenoid valves"
- moved on the sheet: D1, D2, D3, D4, J5, J6, J7, J8, JP1, JP2, JP3, Q1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

Commit message: Brought in test code developed in a different directory
Parts:
- R21, R22: value 47K -> 1.5K
Changed lines of the file:
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@@
 <drawing>
 <settings>
-<setting alwaysvectorfont="yes"/>
+<setting alwaysvectorfont="no"/>
 <setting verticaltext="up"/>
 </settings>
-<grid distance="0.1" unitdist="inch" unit="inch" style="lines" multiple="1" display="no" altdistance="0.01" altunitdist="inch" altunit="inch"/>
+<grid distance="0.1" unitdist="inch" unit="inch" style="lines" multiple="1" display="yes" altdistance="0.01" altunitdist="inch" altunit="inch"/>
 <layers>
 <layer number="1" name="Top" color="4" fill="1" visible="no" active="no"/>
@@
 <part name="JP2" library="AUmlib" library_urn="urn:adsk.eagle:library:9166017" deviceset="PINHD-1X2" device="MOLEX-02-VERT" package3d_urn="urn:adsk.eagle:package:16444314/3" value="MOLEX 53822112022"/>
 <part name="JP3" library="AUmlib" library_urn="urn:adsk.eagle:library:9166017" deviceset="PINHD-1X2" device="MOLEX-02-VERT" package3d_urn="urn:adsk.eagle:package:16444314/3" value="MOLEX 53822112022"/>
-<part name="R21" library="AUmlib" library_urn="urn:adsk.eagle:library:9166017" deviceset="R-US_" device="R0805" package3d_urn="urn:adsk.eagle:package:4021199/4" value="47K"/>
-<part name="R22" library="AUmlib" library_urn="urn:adsk.eagle:library:9166017" deviceset="R-US_" device="R0805" package3d_urn="urn:adsk.eagle:package:4021199/4" value="47K"/>
+<part name="R21" library="AUmlib" library_urn="urn:adsk.eagle:library:9166017" deviceset="R-US_" device="R0805" package3d_urn="urn:adsk.eagle:package:4021199/4" value="1.5K"/>
+<part name="R22" library="AUmlib" library_urn="urn:adsk.eagle:library:9166017" deviceset="R-US_" device="R0805" package3d_urn="urn:adsk.eagle:package:4021199/4" value="1.5K"/>
 <part name="R23" library="AUmlib" library_urn="urn:adsk.eagle:library:9166017" deviceset="R-US_" device="R0805" package3d_urn="urn:adsk.eagle:package:4021199/4" value="1.5K"/>
 <part name="R24" library="AUmlib" library_urn="urn:adsk.eagle:library:9166017" deviceset="R-US_" device="R0805" package3d_urn="urn:adsk.eagle:package:4021199/4" value="1.5K"/>
